File: output/pcbs/board.kicad_pcb (KiCad board)
At the start: 2 copper layers, 183.6 x 137.9 mm, 71 parts

Commit message: As manufactured
Parts:
- added G***: LOGO, LOGO, F.Cu at (73.7, -8.75)
- added TRRS3: TRRS-PJ-320A-dual, TRRS-PJ-320A-dual, F.Cu at (44.4, -78.9)
- added TRRS4: TRRS-PJ-320A-dual, TRRS-PJ-320A-dual, F.Cu at (42.4, -78.9)
- moved B1 93.3 mm to (55.4, 0.00)
- moved TRRS1 1.80 mm to (159.6, -16.8)
- moved TRRS2 1.80 mm to (157.6, -16.8)
- moved D31 1.70 mm to (159.6, 13.6)
- moved D29 1.70 mm to (137.1, 0.67)
- moved D11 1.70 mm to (55.4, -47.7)
- moved D12 1.70 mm to (55.4, -65.3)
- moved D14 1.70 mm to (74.2, -37.0)
- moved D15 1.70 mm to (74.2, -54.7)
- moved D16 1.70 mm to (74.2, -72.3)
- moved D19 1.70 mm to (92.9, -41.7)
- moved D20 1.70 mm to (92.9, -59.3)
- moved D23 1.70 mm to (111.6, -39.2)
- moved D25 1.70 mm to (74.2, 13.9)
- moved D26 1.70 mm to (92.9, 13.9)
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Connections:
- TRRS1 pad 1: VCC -> (no net)
- TRRS1 pad 2: (no net) -> VCC
- TRRS2 pad 1: VCC -> (no net)
- TRRS2 pad 2: (no net) -> VCC
Routing:
- net P3: track 0.00 -> 258.8 mm, vias 0 -> 2
- net P7: track 0.00 -> 258.1 mm, vias 0 -> 2
- net GND: track 0.00 -> 250.5 mm
- net P4: track 0.00 -> 227.6 mm, vias 0 -> 3
- net P5: track 0.00 -> 226.2 mm, vias 0 -> 3
- net P2: track 0.00 -> 224.5 mm, vias 0 -> 3
- net VCC: track 0.00 -> 205.0 mm
- net P10: track 0.00 -> 202.5 mm
- net P19: track 0.00 -> 199.5 mm, vias 0 -> 1
- net P16: track 0.00 -> 194.5 mm
- net P15: track 0.00 -> 183.0 mm
- net P14: track 0.00 -> 182.6 mm
- net P0: track 0.00 -> 182.4 mm
- net P18: track 0.00 -> 181.8 mm
- net P6: track 0.00 -> 177.3 mm, vias 0 -> 1
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Other:
- outline, holes or cut-outs redrawn
- net class Default removed
- net class Power removed
